Commit message: feat: integrate RS06 robot model, validated gait telemetry and scale references

File: ros2_ws/src/robodog_description/urdf/leg.xacro (robot description, xacro)
@@ -21,4 +21,6 @@
     <xacro:property name="tau_max" value="${RS['performance']['peak_torque_nm']}"/>
     <xacro:property name="vel_max" value="${RS['performance']['no_load_speed_rad_s']}"/>
+    <xacro:property name="knee_ratio" value="${RS['transmissions']['kfe']['ratio']}"/>
+    <xacro:property name="knee_efficiency" value="${RS['transmissions']['kfe']['efficiency']}"/>
     <xacro:property name="soft"    value="${OL['position_margin_rad']}"/>
     <xacro:rd_link name="${leg}_hip"   L="${P['links'][leg + '_hip']}"/>
@@ -52,7 +54,7 @@
     </joint>
     <!-- ========== KFE : knee ==========
-         Driven by an actuator mounted proximally on the thigh through a 1:1
+         Driven by an actuator mounted proximally on the thigh through a 2:1
          belt, so the joint stays kinematically simple but the thigh carries the
-         motor mass (COM only 27 mm below the hip) and the calf is just 172 g. -->
+         motor mass; the calf carries the distal structure and foot. -->
     <joint name="${leg}_kfe_joint" type="revolute">
       <parent link="${leg}_thigh"/>
@@ -61,9 +63,9 @@
       <axis xyz="0 1 0"/>
       <limit lower="${JL['kfe']['lower']}" upper="${JL['kfe']['upper']}"
-             effort="${tau_max}" velocity="${vel_max}"/>
+             effort="${tau_max * knee_ratio * knee_efficiency}" velocity="${vel_max / knee_ratio}"/>
       <safety_controller soft_lower_limit="${JL['kfe']['lower'] + soft}"
                          soft_upper_limit="${JL['kfe']['upper'] - soft}"
                          k_position="100.0" k_velocity="10.0"/>
-      <dynamics damping="${JD['damping_nms_per_rad']}" friction="${JD['coulomb_friction_nm']}"/>
+      <dynamics damping="${JD['damping_nms_per_rad'] * knee_ratio * knee_ratio}" friction="${JD['coulomb_friction_nm'] * knee_ratio}"/>
     </joint>
     <!-- ========== foot frame ==========

File: ros2_ws/src/robodog_description/urdf/robodog.urdf.xacro (robot description, xacro)
@@ -2,5 +2,5 @@
 <!--
   =========================================================================
-  robodog - 12-DOF quadruped, 12 x ROBSTRIDE02 QDD actuators, 10 kg target
+  robodog - 12-DOF quadruped, 12 x ROBSTRIDE06 QDD actuators, 19.72 kg working model
   =========================================================================
   Derived from cad/robot/onshape_export by tools/cad_to_model.py. Every number
@@ -8,5 +8,5 @@
   contains no hard-coded geometry.
     config/robot_parameters.yaml  kinematics, inertias, visuals, collisions
-    config/robstride02.yaml       actuator limits, dynamics, CAN scaling
+    config/robstride06.yaml       actuator limits, dynamics, CAN scaling
   Frames (REP-103): x forward, y left, z up. base_link at the body geometric
   centre, which is also within 3.6 mm of the centre of mass.
@@ -31,5 +31,5 @@
   <xacro:property name="PKG" value="$(find robodog_description)"/>
   <xacro:property name="P"   value="${xacro.load_yaml(PKG + '/config/robot_parameters.yaml')}"/>
-  <xacro:property name="RS"  value="${xacro.load_yaml(PKG + '/config/robstride02.yaml')}"/>
+  <xacro:property name="RS"  value="${xacro.load_yaml(PKG + '/config/' + P.get('actuator_config', 'robstride06.yaml'))}"/>
   <xacro:include filename="$(find robodog_description)/urdf/common.xacro"/>
   <xacro:include filename="$(find robodog_description)/urdf/leg.xacro"/>

File: ros2_ws/src/robodog_description/urdf/ros2_control.xacro (robot description, xacro)
@@ -8,5 +8,5 @@
   implement now, and that the C++ SystemInterface plugins must implement when
   the control loop moves into controller_manager.
-  The command interface set is deliberately the ROBSTRIDE02 native impedance
+  The command interface set is deliberately the ROBSTRIDE06 native impedance
   command (position, velocity, effort, kp, kd) rather than a single position
   interface, because that is what the motor accepts on CAN in one frame. Any
@@ -23,11 +23,13 @@
         </xacro:if>
         <xacro:if value="${hardware == 'real'}">
-          <plugin>robodog_hardware/RobStride02CanSystem</plugin>
+          <plugin>robodog_hardware/RobStride06CanSystem</plugin>
           <param name="bus_config">$(find robodog_hardware)/config/robstride_bus.yaml</param>
         </xacro:if>
       </hardware>
       <xacro:macro name="rd_joint_iface" params="jname jkind">
+        <xacro:property name="ratio" value="${RS['transmissions'][jkind]['ratio']}"/>
+        <xacro:property name="efficiency" value="${RS['transmissions'][jkind]['efficiency']}"/>
         <joint name="${jname}">
-          <!-- command: the RS02 motion-control frame, one CAN message -->
+          <!-- command: the RS06 motion-control frame, one CAN message -->
           <command_interface name="position">
             <param name="min">${P['joint_limits'][jkind]['lower']}</param>
@@ -35,14 +37,14 @@
           </command_interface>
           <command_interface name="velocity">
-            <param name="min">${-RS['operational_limits']['velocity_rad_s']}</param>
-            <param name="max">${ RS['operational_limits']['velocity_rad_s']}</param>
+            <param name="min">${-RS['operational_limits']['velocity_rad_s'] / ratio}</param>
+            <param name="max">${ RS['operational_limits']['velocity_rad_s'] / ratio}</param>
           </command_interface>
           <command_interface name="effort">
-            <param name="min">${-RS['performance']['peak_torque_nm']}</param>
-            <param name="max">${ RS['performance']['peak_torque_nm']}</param>
+            <param name="min">${-RS['performance']['peak_torque_nm'] * ratio * efficiency}</param>
+            <param name="max">${ RS['performance']['peak_torque_nm'] * ratio * efficiency}</param>
           </command_interface>
-          <command_interface name="kp"><param name="min">0.0</param><param name="max">500.0</param></command_interface>
-          <command_interface name="kd"><param name="min">0.0</param><param name="max">5.0</param></command_interface>
-          <!-- state: the RS02 feedback frame -->
+          <command_interface name="kp"><param name="min">0.0</param><param name="max">${RS['can']['scaling']['kp_max'] * ratio * ratio * efficiency}</param></command_interface>
+          <command_interface name="kd"><param name="min">0.0</param><param name="max">${RS['can']['scaling']['kd_max'] * ratio * ratio * efficiency}</param></command_interface>
+          <!-- state: the RS06 feedback frame -->
           <state_interface name="position"/>
           <state_interface name="velocity"/>

File: ros2_ws/src/robodog_description/urdf/sensors.xacro (robot description, xacro)
@@ -55,8 +55,9 @@
     <link name="camera_link">
       <inertial>
-        <mass value="0.068"/>
-        <origin xyz="${back} 0 0" rpy="0 0 0"/>
-        <inertia ixx="1.0e-5" ixy="0" ixz="0" iyy="5.0e-5" iyz="0" izz="5.0e-5"/>
+        <mass value="${CM['mass_kg']}"/>
+        <origin xyz="${CM['com_xyz'][0]} ${CM['com_xyz'][1]} ${CM['com_xyz'][2]}" rpy="0 0 0"/>
+        <inertia ixx="${CM['inertia'][0]}" ixy="0" ixz="0" iyy="${CM['inertia'][1]}" iyz="0" izz="${CM['inertia'][2]}"/>
       </inertial>
+      <xacro:unless value="${CM['visual_in_base']}">
       <visual>
         <origin xyz="${back} 0 0" rpy="0 0 0"/>
@@ -68,4 +69,5 @@
         <geometry><box size="${bx} ${by} ${bz}"/></geometry>
       </collision>
+      </xacro:unless>
     </link>
     <joint name="camera_mount_joint" type="fixed">
